File: Hardware/lux-et-pcb/lux-et-pcb.kicad_sch (KiCad schematic)
At the start: 98 parts, among them J1 Conn_01x03_Socket, J2 Conn_01x03_Socket, J3 Conn_01x03_Socket, J4 USB_C_Receptacle_PowerOnly_6P, Q1 PMOS, Q2 PMOS, Q3 AO3400A, Q4 AO3400A, Q5 AO3400A, Q6 2N7002K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

Commit message: Minor update
Other:
- moved on the sheet: C1, C2, D4, PROG1, R1, R4, R6, RST1, U3

Commit message: Current hardware update
Parts:
- removed B2: Conn_01x02_Socket, Connector_Molex:Molex_KK-254_AE-6410-02A_1x02_P2.54mm_Vertical, symbol Connector:Conn_01x02_Socket
- removed C3, C9: 100uF, Capacitor_SMD:C_Elec_6.3x7.7, symbol Device:C_Polarized
- removed D3: 1N4148W, Diode_SMD:D_SOD-123, symbol Diode:1N4148W
- removed NTC1: 10k@25, Connector_PinHeader_1.27mm:PinHeader_1x02_P1.27mm_Vertical, symbol Device:R
- removed Q6: 2N7002K, Package_TO_SOT_SMD:SOT-23, symbol Transistor_FET:2N7002K
- removed R19: 86k6, Resistor_SMD:R_0402_1005Metric, symbol Device:R
- removed R20, R9: 10k, Resistor_SMD:R_0402_1005Metric, symbol Device:R
- removed R23: 0R22, Resistor_SMD:R_1206_3216Metric, symbol Device:R
- removed R24, R25: 2k2, Resistor_SMD:R_0805_2012Metric, symbol Device:R
- added D15, D3: SS14, Diode_SMD:D_SMA, symbol Diode:SS14
- C5, C6: value 100uF -> 220uF; LCSC C99837 -> C7471881
- R10: value 4870 -> 0R22; footprint Resistor_SMD:R_0402_1005Metric -> Resistor_SMD:R_2010_5025Metric; LCSC C25902 -> C2999625
- R14, R15: footprint Resistor_SMD:R_0402_1005Metric -> Resistor_SMD:R_0805_2012Metric
- R18: footprint Resistor_SMD:R_0402_1005Metric -> Resistor_SMD:R_0805_2012Metric; LCSC C25879 -> C17520
- R7: footprint Resistor_SMD:R_0402_1005Metric -> Resistor_SMD:R_0805_2012Metric; LCSC C60491 -> C149504
- renumbered B1 to CC1, SERIAL1 to PORT1, SERIAL2 to PORT2, OLED1 to PORT3
Connections:
- net ButtonA is gone; now on net PCH1: CC1.1 (Pin_1)
- net CE is gone; now on an unnamed net: U4.8 (CE)
- net VTH is gone; now on net GND: R10.1, U4.1 (TEMP)
- net +5V: now also C6.1, D15.1 (K), D3.1 (K); no longer J4.A9 (VBUS), J4.B9 (VBUS), R10.2
- net GND: no longer CC1.2 (Pin_2)
- net NCH1: now also CC1.2 (Pin_2), R10.2
- net VCC: no longer C6.1
- net at PORT1.1 (Pin_1): now also D3.2 (A)
- new net: D15.2 (A), J4.A9 (VBUS), J4.B9 (VBUS)
Other:
- note added: "220mR 700mA"
- note removed: "250mR 620mA"
- note removed: "Buttons"
- moved on the sheet: C1, C2, C7, CC1, D12, D13, PORT2, PROG1, R1, R14, R15, R4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

Commit message: First finished layout for review
Parts:
- removed RV1: R_Potentiometer_Trim, symbol Device:R_Potentiometer_Trim
- J4: footprint Connector_USB:USB_C_Receptacle_GCT_USB4125-xx-x-0190_6P_TopMnt_Horizontal -> Library:USB-C-SMD_GT-USB-7101A
- U3: footprint RF_Module:ESP32-WROOM-32 -> RF_Module:ESP32-WROOM-32U; symbol RF_Module:ESP32-WROOM-32 -> RF_Module:ESP32-WROOM-32U
Connections:
- net CH0: now also U3.16 (IO13)
- net CH1: now also U3.13 (IO14)
- net CH2: now also U3.12 (IO27)
- net CH3: now also U3.11 (IO26)
- net GND: now also U5.4 (FB)
- net WLED_0: now also U3.8 (IO32)
- net WLED_1: now also U3.9 (IO33)
- net WLED_2: now also U3.31 (IO19)
- net WLED_3: now also U3.27 (IO16)
- net IO17: now reaches U3.28 (IO17)
- net IO17: now also PORT2.2 (Pin_2)
- net IO18: now reaches U3.30 (IO18)
- net IO18: now also PORT2.3 (Pin_3)
- net IO2: no longer names the net of U3.24 (IO2)
- net IO2: no longer PORT2.2 (Pin_2)
- net IO4: no longer names the net of U3.26 (IO4)
- net IO4: no longer PORT2.3 (Pin_3)
- no-connect marks 8 -> 9
Other:
- moved on the sheet: C11, CC1, D14, D4, L3, Q7, R10, R22, R26, R6

Commit message: Yet another version for review before fabrication
Parts:
- PORT1, PORT2: footprint Connector_Hirose:Hirose_DF13C_CL535-0404-8-51_1x04-1MP_P1.25mm_Vertical -> Library:Hirose_DF13C_CL535-0404-8-51_1x04-1MP_P1.25mm_Vertical
- PORT3: footprint Connector_Hirose:Hirose_DF13C_CL535-0404-8-51_1x04-1MP_P1.25mm_Vertical -> Library:Hirose_DF13C_CL535-0404-8-51_1x04-1MP_P1.25mm_Vertical; symbol Connector:Conn_01x04_Socket -> New_Library:Conn_01x04_Socket
Connections:
- net CH1: now also U3.12 (IO27); no longer U3.13 (IO14)
- net CH2: now also U3.11 (IO26); no longer U3.12 (IO27)
- net CH3: now also U3.10 (IO25); no longer U3.11 (IO26)
Changed lines of the file:
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@@
 	(wire
 		(pts
-			(xy 251.46 74.93) (xy 248.92 74.93)
-		)
-		(stroke
-			(width 0)
-			(type default)
-		)
-	)
-	(wire
-		(pts
 			(xy 130.81 128.27) (xy 130.81 130.81)
 		)
@@
 	(wire
 		(pts
-			(xy 251.46 49.53) (xy 248.92 49.53)
-		)
-		(stroke
-			(width 0)
-			(type default)
-		)
-	)
-	(wire
-		(pts
 			(xy 207.01 67.31) (xy 207.01 71.12)
 		)
@@
 	(wire
 		(pts
-			(xy 251.46 77.47) (xy 248.92 77.47)
+			(xy 248.92 72.39) (xy 251.46 72.39)
 		)
 		(stroke
@@
 	(wire
 		(pts
+			(xy 248.92 74.93) (xy 251.46 74.93)
+		)
+		(stroke
+			(width 0)
+			(type default)
+		)
+	)
+	(wire
+		(pts
 			(xy 25.4 133.35) (xy 34.29 133.35)
 		)
@@
 	(wire
 		(pts
+			(xy 248.92 77.47) (xy 251.46 77.47)
+		)
+		(stroke
+			(width 0)
+			(type default)
+		)
+	)
+	(wire
+		(pts
 			(xy 90.17 44.45) (xy 90.17 49.53)
 		)
@@
 	(global_label "CH1"
 		(shape input)
-		(at 251.46 49.53 0)
+		(at 251.46 77.47 0)
 		(fields_autoplaced yes)
 		(effects
@@
 		)
 		(property "Intersheetrefs" "${INTERSHEET_REFS}"
-			(at 258.2552 49.53 0)
+			(at 258.2552 77.47 0)
 			(effects
 				(font
@@
 	(global_label "CH2"
 		(shape input)
-		(at 251.46 77.47 0)
+		(at 251.46 74.93 0)
 		(fields_autoplaced yes)
 		(effects
@@
 		)
 		(property "Intersheetrefs" "${INTERSHEET_REFS}"
-			(at 258.2552 77.47 0)
+			(at 258.2552 74.93 0)
 			(effects
 				(font
@@
 	(global_label "CH3"
 		(shape input)
-		(at 251.46 74.93 0)
+		(at 251.46 72.39 0)
 		(fields_autoplaced yes)
 		(effects
@@
 		)
 		(property "Intersheetrefs" "${INTERSHEET_REFS}"
-			(at 258.2552 74.93 0)
+			(at 258.2552 72.39 0)
 			(effects
 				(font
@@
 			)
 		)
-		(property "Footprint" "Connector_Hirose:Hirose_DF13C_CL535-0404-8-51_1x04-1MP_P1.25mm_Vertical"
+		(property "Footprint" "Library:Hirose_DF13C_CL535-0404-8-51_1x04-1MP_P1.25mm_Vertical"
 			(at 261.62 31.75 0)
 			(effects
@@
 			)
 		)
-		(property "Footprint" "Connector_Hirose:Hirose_DF13C_CL535-0404-8-51_1x04-1MP_P1.25mm_Vertical"
+		(property "Footprint" "Library:Hirose_DF13C_CL535-0404-8-51_1x04-1MP_P1.25mm_Vertical"
 			(at 184.15 68.58 0)
 			(effects
@@
 	)
 	(symbol
-		(lib_id "Connector:Conn_01x04_Socket")
+		(lib_id "New_Library:Conn_01x04_Socket")
 		(at 187.96 36.83 0)
 		(unit 1)
@@
 			)
 		)
-		(property "Footprint" "Connector_Hirose:Hirose_DF13C_CL535-0404-8-51_1x04-1MP_P1.25mm_Vertical"
+		(property "Footprint" "Library:Hirose_DF13C_CL535-0404-8-51_1x04-1MP_P1.25mm_Vertical"
 			(at 187.96 36.83 0)
 			(effects
