File: Hardware/lux-et-pcb/lux-et-pcb.kicad_pcb (KiCad board)
At the start: 2 copper layers, 80 x 39 mm, 97 parts, among them J1 Conn_01x03_Socket, J2 Conn_01x03_Socket, J3 Conn_01x03_Socket, J4 USB_C_Receptacle_PowerOnly_6P, Q1 PMOS, Q2 PMOS, Q3 AO3400A, Q4 AO3400A, Q5 AO3400A, Q6 2N7002K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

Commit message: Minor update
Parts:
- moved H1 7.50 mm to (123.8, 56.8)
- moved H2 7.50 mm to (195.8, 56.8)
- moved H3 7.50 mm to (195.8, 102.8)
- moved H4 7.50 mm to (123.8, 102.8)
- moved D10 7.10 mm to (174.0, 56.8)
- moved D5 7.10 mm to (145.5, 56.8)
- moved C1 6.01 mm to (150.2, 83.7)
- moved C2 6.01 mm to (168.5, 83.7)
- moved PROG1 6.01 mm to (163.4, 84.3)
- moved R1 6.01 mm to (170.8, 83.7)
- moved R4 6.01 mm to (148.0, 83.7)
- moved RST1 6.01 mm to (155.4, 84.3)
- moved CD1 6.00 mm to (144.2, 66.4)
- moved CD3 6.00 mm to (146.8, 66.4)
- moved L2 6.00 mm to (145.4, 63.8)
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Routing:
- net PROG: track 13.8 -> 0.00 mm
- net EN: track 10.0 -> 0.00 mm
- net /3V3MCU: track 6.36 -> 1.85 mm
Other:
- board size 80 x 39 mm -> 80 x 54 mm

Commit message: Current hardware update
Parts:
- removed B1, B2: Conn_01x02_Socket, Connector_Molex:Molex_KK-254_AE-6410-02A_1x02_P2.54mm_Vertical
- removed C3, C9: 100uF, Capacitor_SMD:C_Elec_6.3x7.7
- removed NTC1: 10k@25, Connector_PinHeader_1.27mm:PinHeader_1x02_P1.27mm_Vertical
- removed Q6: 2N7002K, Package_TO_SOT_SMD:SOT-23
- removed R19: 86k6, Resistor_SMD:R_0402_1005Metric
- removed R20, R9: 10k, Resistor_SMD:R_0402_1005Metric
- removed R23: 0R22, Resistor_SMD:R_1206_3216Metric
- removed R24, R25: 2k2, Resistor_SMD:R_0805_2012Metric
- added CC1: Conn_01x02_Socket, Connector_Molex:Molex_KK-254_AE-6410-02A_1x02_P2.54mm_Vertical, F.Cu at (165.2, 102.5)
- added D15: SS14, Diode_SMD:D_SMA, F.Cu at (122.5, 94.8)
- C5, C6: value 100uF -> 220uF
- D3: value 1N4148W -> SS14; footprint Diode_SMD:D_SOD-123 -> Diode_SMD:D_SMA
- R10: value 4870 -> 0R22; footprint Resistor_SMD:R_0402_1005Metric -> Resistor_SMD:R_2010_5025Metric
- R14, R15, R18, R7: footprint Resistor_SMD:R_0402_1005Metric -> Resistor_SMD:R_0805_2012Metric
- moved D3 110.9 mm to (188.3, 63.0), turned to 180 degrees
- moved C8 96.6 mm to (187.0, 70.0), turned to -90 degrees
- moved J1 95.1 mm to (195.8, 67.5), turned to 90 degrees
- moved C11 93.7 mm to (172.0, 94.2), turned to 90 degrees
- moved F1 85.3 mm to (173.2, 84.7), turned to -90 degrees
- moved R8 84.4 mm to (179.3, 96.2)
- moved R2 84.1 mm to (172.0, 64.1), turned to -90 degrees
- moved R3 82.0 mm to (172.0, 69.7), turned to 90 degrees
- moved J3 81.6 mm to (180.5, 102.0)
- moved R6 81.0 mm to (174.5, 64.2), turned to -90 degrees
- moved U2 75.8 mm to (158.1, 89.1), turned to 180 degrees
- moved D4 73.9 mm to (174.5, 68.3), turned to 90 degrees
- moved C10 70.0 mm to (141.2, 80.0)
- moved Q2 69.1 mm to (185.9, 87.2), turned to 180 degrees
- moved C6 67.6 mm to (149.2, 91.2), turned to 90 degrees
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- renumbered SERIAL1 to PORT1, SERIAL2 to PORT2, OLED1 to PORT3
Connections:
- C6 pad 1: VCC -> +5V
- J4 pad A9: +5V -> Net-(D15-A)
- J4 pad B9: +5V -> Net-(D15-A)
- R10 pad 1: VTH -> GND
- R10 pad 2: +5V -> NCH1
- R8 pad 2: Net-(U4-VCC) -> Net-(U4-CE)
- U4 pad 1: VTH -> GND
- U4 pad 4: Net-(U4-VCC) -> Net-(U4-CE)
- U4 pad 8: CE -> Net-(U4-CE)
Routing:
- net V_REG: track 0.00 -> 163.7 mm, vias 0 -> 2
- net +5V: track 6.44 -> 91.7 mm, vias 0 -> 4
- net +3.3V: track 1.80 -> 41.9 mm, vias 0 -> 2
- net SCL: track 0.00 -> 34.0 mm, vias 0 -> 2
- net SDA: track 0.00 -> 32.1 mm, vias 0 -> 2
- net VCC: track 31.1 -> 63.2 mm
- net Net-(D8-DOUT): track 0.00 -> 30.2 mm, vias 0 -> 2
- net EN: track 0.00 -> 29.6 mm, vias 0 -> 2
- net Net-(D5-DOUT): track 0.00 -> 24.4 mm, vias 0 -> 2
- net RX0: track 0.00 -> 21.5 mm, vias 0 -> 2
- net Net-(U2-EN): track 0.00 -> 19.7 mm
- net TX0: track 0.00 -> 19.1 mm, vias 0 -> 2
- net +BATT: track 0.00 -> 15.8 mm
- net NCH1: track 0.00 -> 15.5 mm, vias 0 -> 2
- net Net-(U4-CE): track 0.00 -> 14.4 mm, vias 0 -> 2
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Other:
- outline, holes or cut-outs redrawn

Commit message: First finished layout for review
Parts:
- J4: footprint Connector_USB:USB_C_Receptacle_GCT_USB4125-xx-x-0190_6P_TopMnt_Horizontal -> Library:USB-C-SMD_GT-USB-7101A
- U3: footprint RF_Module:ESP32-WROOM-32 -> RF_Module:ESP32-WROOM-32U
- moved J1 60.4 mm to (136.2, 57.2), turned to 180 degrees
- moved J2 60.4 mm to (195.8, 67.5), turned to 90 degrees
- moved R3 20.7 mm to (191.5, 76.7)
- moved J4 0.72 mm to (122.7, 85.0)
- moved VDC1 0.49 mm to (128.5, 72.7)
Connections:
- PORT2 pad 2: IO2 -> IO17
- PORT2 pad 3: IO4 -> IO18
- U3 pad 11: unconnected-(U3-IO26-Pad11) -> CH3
- U3 pad 12: unconnected-(U3-IO27-Pad12) -> CH2
- U3 pad 13: unconnected-(U3-IO14-Pad13) -> CH1
- U3 pad 16: unconnected-(U3-IO13-Pad16) -> CH0
- U3 pad 24: IO2 -> unconnected-(U3-IO2-Pad24)
- U3 pad 26: IO4 -> unconnected-(U3-IO4-Pad26)
- U3 pad 27: unconnected-(U3-IO16-Pad27) -> WLED_3
- U3 pad 28: unconnected-(U3-IO17-Pad28) -> IO17
- U3 pad 30: unconnected-(U3-IO18-Pad30) -> IO18
- U3 pad 31: unconnected-(U3-IO19-Pad31) -> WLED_2
- U3 pad 8: unconnected-(U3-IO32-Pad8) -> WLED_0
- U3 pad 9: unconnected-(U3-IO33-Pad9) -> WLED_1
- U5 pad 4: Net-(U5-FB) -> GND
Routing:
- net +3.3V: track 41.9 -> 173.1 mm, vias 2 -> 9
- net V_REG: track 163.7 -> 263.3 mm, vias 2 -> 8
- net +5V: track 91.7 -> 158.8 mm, vias 4 -> 19
- net WLED_3: track 0.00 -> 56.6 mm, vias 0 -> 3
- net Net-(D6-DOUT): track 0.00 -> 50.4 mm, vias 0 -> 2
- net WLED_1: track 0.00 -> 40.5 mm, vias 0 -> 1
- net Net-(D10-DIN): track 0.00 -> 40.4 mm, vias 0 -> 2
- net WLED_2: track 0.00 -> 34.2 mm, vias 0 -> 2
- net IO18: track 0.00 -> 31.8 mm, vias 0 -> 2
- net IO17: track 0.00 -> 31.3 mm, vias 0 -> 2
- net CH0: track 2.00 -> 30.0 mm, vias 0 -> 2
- net CH3: track 0.00 -> 26.9 mm, vias 0 -> 2
- net Net-(D7-DOUT): track 0.00 -> 26.2 mm, vias 0 -> 2
- net CH2: track 0.00 -> 24.8 mm, vias 0 -> 2
- net CH1: track 0.00 -> 21.3 mm, vias 0 -> 2
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Other:
- outline, holes or cut-outs redrawn

Commit message: Yet another version for review before fabrication
Parts:
- PORT1, PORT2, PORT3: footprint Connector_Hirose:Hirose_DF13C_CL535-0404-8-51_1x04-1MP_P1.25mm_Vertical -> Library:Hirose_DF13C_CL535-0404-8-51_1x04-1MP_P1.25mm_Vertical
- moved Strip1 34.3 mm to (124.5, 70.7), turned to 90 degrees
- moved Q5 33.7 mm to (130.9, 62.9), turned to 180 degrees
- moved R21 30.7 mm to (134.5, 62.9), turned to 90 degrees
- moved Q4 29.1 mm to (130.9, 67.2), turned to 180 degrees
- moved R17 26.5 mm to (136.8, 63.0)
- moved R16 25.6 mm to (134.5, 67.3), turned to 90 degrees
- moved Q3 25.4 mm to (131.0, 71.2), turned to 180 degrees
- moved R13 21.7 mm to (136.8, 67.3)
- moved R12 21.5 mm to (134.5, 71.3), turned to 90 degrees
- moved J4 20.7 mm to (133.4, 102.8), turned to 0 degrees
- moved R5 20.5 mm to (123.0, 74.7)
- moved VDC1 19.1 mm to (128.7, 91.8)
- moved Q1 18.9 mm to (125.2, 82.3), turned to 180 degrees
- moved D1 18.1 mm to (123.8, 77.1), turned to 180 degrees
- moved C5 18.1 mm to (134.7, 88.3), turned to 180 degrees
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Connections:
- U3 pad 10: unconnected-(U3-IO25-Pad10) -> CH3
- U3 pad 11: CH3 -> CH2
- U3 pad 12: CH2 -> CH1
- U3 pad 13: CH1 -> unconnected-(U3-IO14-Pad13)
Routing:
- net Net-(D6-DOUT): track 50.4 -> 28.0 mm
- net VCC: track 63.1 -> 73.0 mm
- net Net-(D15-A): track 15.7 -> 7.16 mm, vias 2 -> 0
- net +5V: track 158.8 -> 150.6 mm, vias 19 -> 18
- net CH2: track 24.8 -> 17.8 mm, vias 2 -> 0
- net CH3: track 26.9 -> 20.6 mm, vias 2 -> 0
- net CH1: track 21.3 -> 17.3 mm, vias 2 -> 0
- net V_REG: track 263.3 -> 265.5 mm, vias 8 -> 10
- net Net-(Q5-G): track 6.65 -> 4.82 mm
- net R_CH: track 5.64 -> 6.84 mm
- net Net-(Q4-G): track 5.82 -> 4.82 mm
- net Net-(Q3-G): track 5.81 -> 4.81 mm
- net GND: track 3.39 -> 2.49 mm, vias 57 -> 64
- net Vin: track 6.53 -> 7.34 mm
- net B_CH: track 6.36 -> 5.60 mm
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
Commit message: Updated fabrication files
Other:
- board text added: "+ VDC -"
- board text added: "+CC-"
- board text added: "+RGB"
- board text added: "-B+"
- board text added: "-CH1+"
- board text added: "-CH2+"
- board text added: "-CH3+"
Changed lines of the file:
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@@
 		(layer "Edge.Cuts")
 	)
+	(gr_text "-CH3+"
+		(at 185.9 105.3 0)
+		(layer "B.SilkS")
+		(effects
+			(font
+				(size 1 1)
+				(thickness 0.1)
+			)
+			(justify left bottom mirror)
+		)
+	)
+	(gr_text "-CH2+"
+		(at 198.6 62.2 90)
+		(layer "B.SilkS")
+		(effects
+			(font
+				(size 1 1)
+				(thickness 0.1)
+			)
+			(justify left bottom mirror)
+		)
+	)
+	(gr_text "+CC-"
+		(at 166.05 105.23 0)
+		(layer "B.SilkS")
+		(effects
+			(font
+				(size 1 1)
+				(thickness 0.1)
+			)
+			(justify left bottom mirror)
+		)
+	)
+	(gr_text "+\nVDC\n-"
+		(at 125.4 87.7 270)
+		(layer "B.SilkS")
+		(effects
+			(font
+				(size 2 2)
+				(thickness 0.1)
+			)
+			(justify mirror)
+		)
+	)
+	(gr_text "+RGB"
+		(at 120.6 71.9 270)
+		(layer "B.SilkS")
+		(effects
+			(font
+				(size 2 2.3)
+				(thickness 0.1)
+			)
+			(justify left bottom mirror)
+		)
+	)
+	(gr_text "-B+"
+		(at 198.6 93.2 90)
+		(layer "B.SilkS")
+		(effects
+			(font
+				(size 1 1)
+				(thickness 0.1)
+			)
+			(justify left bottom mirror)
+		)
+	)
+	(gr_text "-CH1+"
+		(at 130.9 54.2 180)
+		(layer "B.SilkS")
+		(effects
+			(font
+				(size 1 1)
+				(thickness 0.1)
+			)
+			(justify left bottom mirror)
+		)
+	)
 	(segment
 		(start 168.5 84.5775)
@@
 		)
 	)
-	(group ""
+	(group "HORSE"
 		(members "000b15ba-364d-4643-b227-adc6e7a1135b" "001ca044-84aa-436d-8bff-f56c5bce3069"
 			"002db23c-ba51-4657-b013-b7a4cbaf01b6" "0031402c-758a-4f64-af85-902a6e02b6ab"

Commit message: BoM update
Parts:
- removed J4: USB_C_Receptacle_PowerOnly_6P, Library:USB-C-SMD_GT-USB-7101A
- added J5: USB_C_Receptacle_USB2.0_8P, Library:USB-C-SMD_GT-USB-7101A, F.Cu at (133.4, 102.8)

Commit message: Hardware update
Parts:
- R11, R13, R17, R6: value 330 -> 330R
- R14, R15: value 1k -> 2.2k
- R18, R2, R3: value 2k2 -> 2.2k
- U5: value ~ -> XL4001
Changed lines of the file:
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@@
 			)
 		)
-		(property "Value" "1k"
+		(property "Value" "2.2k"
 			(at 0 1.65 90)
 			(layer "F.Fab")
@@
 			)
 		)
-		(property "LCSC" "C11702"
+		(property "LCSC" "C17520"
 			(at 0 0 -90)
 			(unlocked yes)
@@
 			)
 		)
-		(property "Sim.Pins" "1=D 2=G 3=S"
+		(property "Sim.Pins" "1=G 2=D 3=S"
 			(at 0 0 180)
 			(unlocked yes)
@@
 			)
 		)
-		(property "Value" "~"
+		(property "Value" "XL4001"
 			(at -0.325 4.2085 90)
 			(layer "F.Fab")
@@
 			)
 		)
-		(property "Value" "330"
+		(property "Value" "330R"
 			(at 0 1.65 90)
 			(layer "F.Fab")
@@
 			)
 		)
-		(property "Value" "330"
+		(property "Value" "330R"
 			(at 0 1.65 90)
 			(layer "F.Fab")
@@
 			)
 		)
-		(property "Value" "330"
+		(property "Value" "330R"
 			(at 0 1.65 90)
 			(layer "F.Fab")
@@
 			)
 		)
-		(property "Value" "2k2"
+		(property "Value" "2.2k"
 			(at 0 1.65 0)
 			(layer "F.Fab")
@@
 			)
 		)
-		(property "Value" "2k2"
+		(property "Value" "2.2k"
 			(at 0 1.65 90)
 			(layer "F.Fab")
@@
 			)
 		)
-		(property "Value" "1k"
+		(property "Value" "2.2k"
 			(at 0 1.65 90)
 			(layer "F.Fab")
@@
 			)
 		)
-		(property "LCSC" "C11702"
+		(property "LCSC" "C17520"
 			(at 0 0 -90)
 			(unlocked yes)
@@
 			)
 		)
-		(property "Value" "2k2"
+		(property "Value" "2.2k"
 			(at 0 1.65 90)
 			(layer "F.Fab")
@@
 			)
 		)
-		(property "Value" "330"
+		(property "Value" "330R"
 			(at 0 1.65 90)
 			(layer "F.Fab")
