File: Hardware/lux-et-pcb-V2/lux-et-pcb-V2.kicad_sch (KiCad schematic)
At the start: 88 parts, among them J1 Conn_01x03_Socket, J2 Conn_01x03_Socket, J3 Conn_01x03_Socket, J4 USB_C_Receptacle_PowerOnly_6P, Q1 PMOS, Q2 PMOS, Q3 AO3400A, Q4 AO3400A, Q5 AO3400A, Q7 2N7002K, U1 XL1509-5V, U2 AP2112K-3.3, U3 ESP32-WROOM-32, U4 TP4056

Commit message: Hardware update
Parts:
- added BOOT1: SW_Push, Button_Switch_SMD:SW_SPST_PTS647_Sx38, symbol Switch:SW_Push
- added Q6: 2N7002K, Package_TO_SOT_SMD:SOT-23, symbol Transistor_FET:2N7002K
- added R19, R9: 100k, Resistor_SMD:R_0805_2012Metric, symbol Device:R
- added R20: 10k, Resistor_SMD:R_0805_2012Metric, symbol Device:R
Connections:
- net GND: now also Q6.2 (S), R19.2; no longer U1.4 (~{EN})
- net VCC: now also BOOT1.2, R9.1
- net at D16.1 (K): now also R20.1
- net LATCH: now reaches D16.2 (A)
- net LATCH: now also U3.26 (IO4)
- new net: Q6.3 (D), R9.2, U1.4 (~{EN})
- new net P_ON: BOOT1.1, Q6.1 (G), R19.1, R20.2
Other:
- moved on the sheet: C4, C5, C6, CD2, CD3, D1, D16, D2, F1, L1, L2, Q1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

Commit message: Added V2 base sketch
Parts:
- removed C1, C2: 100n, Capacitor_SMD:C_0805_2012Metric, symbol Device:C
- removed C10, C11: 220uF, Capacitor_SMD:C_Elec_6.3x7.7, symbol Device:C_Polarized
- removed C7: 10u, Capacitor_SMD:C_0805_2012Metric, symbol Device:C
- removed CC1: Conn_01x02_Socket, Connector_Molex:Molex_KK-254_AE-6410-02A_1x02_P2.54mm_Vertical, symbol Connector:Conn_01x02_Socket
- removed D1: D_Zener, Diode_SMD:D_MiniMELF, symbol Device:D_Zener
- removed D12: LED_BLUE, LED_SMD:LED_0805_2012Metric_Pad1.15x1.40mm_HandSolder, symbol Device:LED
- removed D13: LED_RED, LED_SMD:LED_0805_2012Metric_Pad1.15x1.40mm_HandSolder, symbol Device:LED
- removed D14, D15: SS14, Diode_SMD:D_SMA, symbol Diode:SS14
- removed D4: LED, LED_SMD:LED_0805_2012Metric_Pad1.15x1.40mm_HandSolder, symbol Device:LED
- removed J3: Conn_01x03_Socket, TerminalBlock:TerminalBlock_Xinya_XY308-2.54-3P_1x03_P2.54mm_Horizontal, symbol Connector:Conn_01x03_Socket
- removed J4: USB_C_Receptacle_PowerOnly_6P, symbol Connector:USB_C_Receptacle_PowerOnly_6P
- removed L3: 33u, Inductor_SMD:L_Sunlord_SWPA4010S, symbol Device:L
- removed PROG1, RST1: SW_Push, Button_Switch_SMD:SW_SPST_PTS647_Sx38, symbol Switch:SW_Push
- removed Q7: 2N7002K, Package_TO_SOT_SMD:SOT-23, symbol Transistor_FET:2N7002K
- removed R1, R22, R26, R4: 10k, Resistor_SMD:R_0805_2012Metric, symbol Device:R
- removed R10, R8: 0R22, Resistor_SMD:R_2010_5025Metric, symbol Device:R
- removed R14, R15, R18: 2k2, Resistor_SMD:R_0805_2012Metric, symbol Device:R
- removed R27, R28: 5.1k, Resistor_SMD:R_0805_2012Metric, symbol Device:R
- removed U3: ESP32-WROOM-32, RF_Module:ESP32-WROOM-32U, symbol RF_Module:ESP32-WROOM-32U
- removed U4: TP4056, Library:SOP-8_L4.9-W3.9-P1.27-LS6.0-BL-EP, symbol New_Library:TP4056
- removed U5: ~, Library:ESOP-8_L4.9-W3.9-P1.27-LS6.0-BL-EP, symbol New_Library:XL4001E1_C2988027
- added C15, C16: 100nF, Capacitor_SMD:C_0805_2012Metric, symbol Device:C
- added C3: 220uF, Capacitor_SMD:C_Elec_6.3x7.7, symbol Device:C_Polarized
- added PROG2, RST2: SW_Push, Button_Switch_SMD:SW_SPST_PTS647_Sx38, symbol Switch:SW_Push
- added R29, R30, R31, R32: 10k, Resistor_SMD:R_0805_2012Metric, symbol Device:R
- added U7: ESP32-S3-MINI-2, PCM_Espressif:ESP32-S3-MINI-1, symbol PCM_Espressif:ESP32-S3-MINI-1
- C8: value 100uF -> 220uF; LCSC C99837 -> C7471881
- Q1, Q2: LCSC C2593 -> C42456992
- R6: value 330 -> 100k; LCSC C17630 -> C149504
- renumbered CD2 to C2, CD3 to C3, CD4 to C4, CD5 to C5, CD6 to C6, CD7 to C7, CD8 to C8, CD9 to C9
Connections:
- net +3.3V: now also R29.2, R30.1; no longer R6.1
- net +5V: now also C3.1
- net 3V3MCU: now also U7.3 (3V3)
- net EN: now also C15.1, R29.1, RST2.2, U7.45 (EN)
- net GND: now also C15.2, C16.2, C3.2, PROG2.1, R31.2, R32.2, RST2.1, U7.1 (GND), U7.2 (GND), U7.42 (GND), U7.43 (GND), U7.46 (GND), U7.47 (GND), U7.48 (GND), U7.49 (GND), U7.50 (GND), U7.51 (GND), U7.52 (GND), U7.53 (GND), U7.54 (GND), U7.55 (GND), U7.56 (GND), U7.57 (GND), U7.58 (GND), U7.59 (GND), U7.60 (GND), U7.61 (GND), U7.62 (GND), U7.63 (GND), U7.64 (GND), U7.65 (GND)
- net PROG: now also C16.1, PROG2.2, R30.2, U7.4 (GPIO0/BOOT)
- net RX0: now also U7.40 (U0RXD/GPIO44/CLK_OUT2)
- net SCL: now also U7.12 (GPIO8/TOUCH8/ADC1_CH7/SUBSPICS1)
- net SDA: now also U7.11 (GPIO7/TOUCH7/ADC1_CH6)
- net TX0: now also U7.39 (U0TXD/GPIO43/CLK_OUT1)
- net VCC: now also R6.2
- net at Q1.2 (G), R5.1: now also R6.1
- new net: R31.1, U7.41 (GPIO45)
- new net: R32.1, U7.44 (GPIO46)
- new net CLK: U7.32 (SPIIO7/GPIO36/FSPICLK/SUBSPICLK)
- new net CMD: U7.31 (SPIIO6/GPIO35/FSPID/SUBSPID)
- new net DAT0: U7.33 (SPIDQS/GPIO37/FSPIQ/SUBSPIQ)
- new net D_N: U7.23 (GPIO19/U1RTS/ADC2_CH8/CLK_OUT2/USB_D-)
- new net D_P: U7.24 (GPIO20/U1CTS/ADC2_CH9/CLK_OUT1/USB_D+)
- new net SPK: U7.6 (GPIO2/TOUCH2/ADC1_CH1)
- new net SPK_OFF: U7.5 (GPIO1/TOUCH1/ADC1_CH0)
- no-connect marks 9 -> 1
Other:
- added sheet Aditional modules (modules.kicad_sch)
- note added: "/2"
- note added: "External WLED"
- note removed: "220mR 700mA"
- note removed: "CC Driver"
- note removed: "Charger"
- note removed: "ESP32-Wroom"
- note removed: "To do: *Add enable (power saving) *USB-C 6 pin (cheaper) *0402 footprints (smaller)"
- note removed: "WLED"
- moved on the sheet: C2, D16, J1, J2, PORT2, Q3, Q4, Q5, R11, R12, R13, R16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
