File: Hardware/Marajoara_PCB/Marajoara_PCB.kicad_pcb (KiCad board)
At the start: 2 copper layers, 239.5 x 192.5 mm, 97 parts, among them J1 Conn_01x03_Socket, Q1 PMOS, Q2 2N7002K, U1 TP4056, U2 ESP32-C3-Supermini

Commit message: Fabricated PCB files
Parts:
- added C34: 220uF, Capacitor_SMD:CP_Elec_6.3x7.7, F.Cu at (226.5, 148.6)
- added REF**: 18650-1S, Aleoexpress:18650-1S, F.Cu at (182.1, 110.1)
- added VDD1: Conn_01x02_Socket, Connector_Molex:Molex_KK-254_AE-6410-02A_1x02_P2.54mm_Vertical, F.Cu at (156.0, 86.3)
- D10, D11, D12, D27, D28, D3, D4, D5, D6, D7, D8, D9: moved to F.Cu
- Q1: value PMOS -> XR5P04
- moved SPK_L 168.0 mm to (292.6, 93.5)
- moved SPK_R 165.9 mm to (131.2, 93.6)
- moved R10 91.0 mm to (176.4, 101.1)
- moved C28 31.1 mm to (207.8, 211.7), turned to 180 degrees
- moved C29 19.6 mm to (223.0, 214.1), turned to -45 degrees
- moved C25 15.2 mm to (218.5, 183.2), turned to -135 degrees
- moved C33 12.7 mm to (217.8, 205.7), turned to 0 degrees
- moved C32 12.6 mm to (203.8, 205.8), turned to 0 degrees
- moved C31 12.4 mm to (218.4, 195.1), turned to 180 degrees
- moved C30 11.7 mm to (202.5, 195.8)
- moved C27 11.6 mm to (204.8, 183.0), turned to -45 degrees
- moved D7 11.0 mm to (243.5, 196.0), turned to 45 degrees
- moved D8 10.9 mm to (173.1, 193.5), turned to 0 degrees
- moved D9 10.5 mm to (146.2, 171.5)
- moved D5 10.0 mm to (297.5, 146.4)
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Routing:
- net Net-(Q1-G): track 101.1 -> 5.28 mm
- net Net-(D7-DOUT): track 10.1 -> 89.2 mm
- net GND: track 7.66 -> 59.9 mm, vias 93 -> 132
- net V_REG: track 900.8 -> 943.0 mm
- net Net-(D18-DOUT): track 183.2 -> 168.9 mm
- net +5V: track 45.5 -> 58.0 mm
- net +BATT: track 138.1 -> 145.1 mm
- net Net-(D11-DOUT): track 94.0 -> 87.7 mm
- net Net-(D3-DOUT): track 93.4 -> 87.8 mm
- net Button_GPIO: track 106.3 -> 110.7 mm
- net Net-(D32-K): track 105.6 -> 110.0 mm
- net Net-(D26-DOUT): track 10.9 -> 6.68 mm
- net Net-(D24-DOUT): track 12.9 -> 9.98 mm
- net Net-(D10-DIN): track 35.9 -> 33.7 mm
- net Net-(D27-DOUT): track 11.3 -> 9.48 mm
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Other:
- board size 239.5 x 192.5 mm -> 231.3 x 182.5 mm
