File: Hardware/Marajoara_PCB/Marajoara_PCB.kicad_sch (KiCad schematic)
At the start: 91 parts, among them J1 Conn_01x03_Socket, Q1 PMOS, Q2 2N7002K, U1 TP4056, U2 ESP32-C3-Supermini

Commit message: Marajoara update
Parts:
- added H1, H2, H3, H4: MountingHole, MountingHole:MountingHole_3.2mm_M3, symbol Mechanical:MountingHole
- R3: value 0R22 -> 220mR 1W 1%; footprint Resistor_SMD:R_2010_5025Metric -> Resistor_SMD:R_1206_3216Metric_Pad1.30x1.75mm_HandSolder; LCSC C2999625 -> C2683384; Mfr. Part Number (none) -> RLH12FTCR220
Connections:
- net +5V: now also U1.8 (CE); no longer C11.2, C12.2, C13.2, C14.2, C15.2, C16.2, C17.2, C19.2, C20.2, C21.2, C22.2, C23.2, C24.2, C25.2, C27.2, C28.2, C29.2, C3.2, C30.2, C31.2, C32.2, C33.2, C4.2, C5.2, C6.2, C7.2, C8.2, C9.2, D1.3 (VDD), D10.3 (VDD), D11.3 (VDD), D12.3 (VDD), D13.3 (VDD), D14.3 (VDD), D15.3 (VDD), D16.3 (VDD), D17.3 (VDD), D18.3 (VDD), D19.3 (VDD), D2.3 (VDD), D20.3 (VDD), D21.3 (VDD), D22.3 (VDD), D23.3 (VDD), D24.3 (VDD), D25.3 (VDD), D26.3 (VDD), D27.3 (VDD), D28.3 (VDD), D3.3 (VDD), D4.3 (VDD), D5.3 (VDD), D6.3 (VDD), D7.3 (VDD), D8.3 (VDD), D9.3 (VDD)
- net V_REG: now also C11.2, C12.2, C13.2, C14.2, C15.2, C16.2, C17.2, C19.2, C20.2, C21.2, C22.2, C23.2, C24.2, C25.2, C27.2, C28.2, C29.2, C3.2, C30.2, C31.2, C32.2, C33.2, C4.2, C5.2, C6.2, C7.2, C8.2, C9.2, D1.3 (VDD), D10.3 (VDD), D11.3 (VDD), D12.3 (VDD), D13.3 (VDD), D14.3 (VDD), D15.3 (VDD), D16.3 (VDD), D17.3 (VDD), D18.3 (VDD), D19.3 (VDD), D2.3 (VDD), D20.3 (VDD), D21.3 (VDD), D22.3 (VDD), D23.3 (VDD), D24.3 (VDD), D25.3 (VDD), D26.3 (VDD), D27.3 (VDD), D28.3 (VDD), D3.3 (VDD), D4.3 (VDD), D5.3 (VDD), D6.3 (VDD), D7.3 (VDD), D8.3 (VDD), D9.3 (VDD)
- net at R3.2, U1.4 (VCC): no longer U1.8 (CE)

Commit message: Fabricated PCB files
Parts:
- removed Q1: PMOS, Package_TO_SOT_SMD:SOT-23_Handsoldering, symbol Simulation_SPICE:PMOS
- added C34: 220uF, Capacitor_SMD:CP_Elec_6.3x7.7, symbol Device:C_Polarized
- added Q1: XR5P04, Package_TO_SOT_SMD:SOT-23_Handsoldering, symbol ALeoExpress:XR5P04
- added VDD1: Conn_01x02_Socket, Connector_Molex:Molex_KK-254_AE-6410-02A_1x02_P2.54mm_Vertical, symbol Connector:Conn_01x02_Socket
Connections:
- net +5V: now also VDD1.1 (Pin_1)
- net +BATT: now also Q1.2 (S)
- net GND: now also C34.2, VDD1.2 (Pin_2)
- net V_REG: now also C34.1, Q1.3 (D)
- net at Q2.3 (D), R10.1: now also Q1.1 (G)
Other:
- note added: "5V Header"
- moved on the sheet: BATT1, BT1, C1, C10, C11, C12, C13, C14, C15, C16, C17, C18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
