File: Hardware/Marajoara_V2/Marajoara_V2.kicad_sch (KiCad schematic)
At the start: 141 parts, among them J1 Conn_01x03_Socket, J2 USB_C_Receptacle_USB2.0_8P, J3 Conn_01x02_Socket, J4 Conn_01x02_Socket, Q1 PMOS, Q10 2N7002K, Q2 2N7002K, Q3 PMOS, Q9 2N7002K, U1 TP4056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

Commit message: Added Echoes of Termina base firmware
Parts:
- U4, U7: LCSC (none) -> C910544; Link (none) -> https://pt.aliexpress.com/item/1005007852632407.html
Connections:
- net ADC1_0 is gone; now on net ADC1_6: C26.2, R14.1, R15.1
- net ADC1_6: now reaches U13.9 (VDET_1/GPIO34/ADC1_CH6)
- net I2S_DIN renamed I2S_DOUT
Other:
- moved on the sheet: C34, C35, J3, J4, U4, U7
