File: Hardware/lux-et-portabilis-V2/lux-et-portabilis-V2.kicad_sch (KiCad schematic)
At the start: 48 parts, among them J1 Conn_01x03_Socket, J2 Conn_01x03_Socket, J3 Conn_01x04_Socket, Q2 2N7002K, Q3 PMOS, U1 ESP32-C3-Supermini, U2 TP4056

Commit message: Hardware: add clamp diode D7 to the Portabilis V2 button node
D7 - BZV55B2V7, 2.7 V / 500 mW / 2%, zener, MiniMELF
(Diode_SMD:D_MiniMELF) - placed on the Button_GPIO net with a GND return. That
node is the clamp the TOUCH1 / BT1 input is missing: BT1 puts +BATT (~4.2 V) onto
a 3.3 V GPIO through R12, and D6 is not a clamp there because its far end lands
on the latch-gate node instead of a 3.3 V rail. This is the most likely cause of
the touch input that reads LOW on the bench board while its pad measures a clean
3.3 V.

The value is recorded as drawn, not as it should be: the C3's VIH is ~2.48 V, so
a 2.7 V zener sits too close to the logic threshold. 3.3 V or 3.6 V is the part
this node wants.

Schematic only - lux-et-portabilis-V2.kicad_pcb and the production files were not
regenerated for D7, so do not order boards expecting the clamp.

lux_et_portabilis.kicad_prl only flips KiCad's integration_disabled flag back to
false: editor state, no design change.
Parts:
- added D7: BZV55B2V7, Diode_SMD:D_MiniMELF, symbol Diode:BZV55B2V7
Connections:
- net Button_GPIO: now also D7.1 (K)
- net GND: now also D7.2 (A)
Other:
- note added: "Warning: 4.2V fries the button GPIO"
